File: PSE_RP2040/PSE_RP2040.sch (KiCad schematic (older format))
At the start: 16 parts, among them IC1 AT25SF128A-SHB-T, U1 RP2040

Commit message: Modifica schema kicad
Aggiunti librerie, datasheet e componenti
Parts:
- added C1, C2: 47u, symbol Device:C
- added C10, C11, C15, C6, C7, C8, C9, C?: 100n, symbol Device:C
- added C12, C14, C18: 2u2, symbol Device:C
- added C?: 1u, symbol Device:C
- added D?: LED, symbol Device:LED
- added D? (x2): MBR1020VL, Diode_SMD:D_SOD-123F, symbol Diode:MBR1020VL
- added J?: Conn_01x03, symbol Connector_Generic:Conn_01x03
- added L2: 2U2, symbol Device:L
- added Q?: DTC114Y, symbol Transistor_BJT:DTC114Y
- added R11: 1k, symbol Device:R
- added R12, R13: 27, symbol Device:R
- added R2, R8: 100k, symbol Device:R
- added R3: R, symbol Device:R
- added R?: R4 no fit, symbol Device:R
- added R?: 11K, symbol Device:R
- added SW?: SW_Push, symbol Switch:SW_Push
- added U?: MCP1703A-3302_SOT23, Package_TO_SOT_SMD:SOT-23, symbol Regulator_Linear:MCP1703A-3302_SOT23
- added U?: W25Q16JVUXIQ, symbol Flash_memory:W25Q16JVUXIQ
- added U?: PAM7Q, symbol gpsChip:PAM7Q
- added U?: RT6150A_B, symbol buck_converter:RT6150A_B
- gave numbers to parts that had none: 13
Connections:
- net labels added: +1V1, +3.3V, GPIO10, GPIO11, GPIO12, GPIO13, GPIO14, GPIO15, GPIO16, GPIO17, GPIO18, GPIO19, GPIO2, GPIO20, GPIO21, GPIO22, GPIO23, GPIO24, GPIO25, GPIO3, GPIO4, GPIO5, GPIO6, GPIO7, GPIO8, GPIO9, GPS_RESET, PPS, QSPI_SCLK, QSPI_SD0, QSPI_SD1, QSPI_SD2, QSPI_SD3, QSPI_SS, SHUT_DOWN, SWCLK, SWDIO, UART_RX-GPS_TX, UART_TX-GPS_RX
- net labels removed: HOLD, SCK, SERIAL_INPUT, SERIAL_OUTPUT, WRITE_PROTECT
- wire segments 57 -> 216
- no-connect marks 1 -> 2
Other:
- note added: "Alimentazione\n"
- note added: "Localizzazione"
- note added: "Microcontrollore\n"
- note removed: "GPS"
- moved on the sheet: C1, C2, C5, F1, IC1, IC2, J3, R1, R2, R3, U1

Commit message: Modifica quarzo
Parts:
- removed F1: ABLS-12.000MHZ-B4-T, HC/49US-(AT49)_1, symbol PSE_RP2040-rescue:ABLS-12.000MHZ-B4-T-ABLS-12.000MHZ-B4-T_crystal
- added Y?: Crystal_GND24, symbol Device:Crystal_GND24
- C2, C5: value 27p -> ?
- U?: symbol Flash_memory:W25Q16JVUXIQ -> PSE_RP2040-rescue:W25Q16JVUXIQ-Flash_memory
- U?: symbol gpsChip:PAM7Q -> PSE_RP2040-rescue:PAM7Q-gpsChip
- U?: symbol buck_converter:RT6150A_B -> PSE_RP2040-rescue:RT6150A_B-buck_converter
Connections:
- wire segments 216 -> 219
Changed lines of the file:
@@
 EESchema Schematic File Version 4
-LIBS:PSE_RP2040-cache
 EELAYER 30 0
 EELAYER END
@@
 QSPI_SD3
 $Comp
-L PSE_RP2040-rescue:ABLS-12.000MHZ-B4-T-ABLS-12.000MHZ-B4-T_crystal F1
-U 1 1 622EB81D
-P 4100 3550
-F 0 "F1" H 4450 3775 50  0000 C CNN
-F 1 "ABLS-12.000MHZ-B4-T" H 4450 3684 50  0000 C CNN
-F 2 "HC/49US-(AT49)_1" H 4650 3600 50  0001 L CNN
-F 3 "https://componentsearchengine.com/Datasheets/2/ABLS-12.000MHZ-B4-T.pdf" H 4650 3500 50  0001 L CNN
-F 4 "ABRACON - ABLS-12.000MHZ-B4-T - CRYSTAL, 12MHZ, 18PF, HC-49US" H 4650 3400 50  0001 L CNN "Description"
-F 5 "" H 4650 3300 50  0001 L CNN "Height"
-F 6 "ABRACON" H 4650 3200 50  0001 L CNN "Manufacturer_Name"
-F 7 "ABLS-12.000MHZ-B4-T" H 4650 3100 50  0001 L CNN "Manufacturer_Part_Number"
-F 8 "815-ABLS-12.0M-T" H 4650 3000 50  0001 L CNN "Mouser Part Number"
-F 9 "https://www.mouser.co.uk/ProductDetail/ABRACON/ABLS-12000MHZ-B4-T?qs=yTU0IcKoRlGSQ8ooxPPVnQ%3D%3D" H 4650 2900 50  0001 L CNN "Mouser Price/Stock"
-F 10 "ABLS-12.000MHZ-B4-T" H 4650 2800 50  0001 L CNN "Arrow Part Number"
-F 11 "https://www.arrow.com/en/products/abls-12.000mhz-b4-t/abracon?region=nac" H 4650 2700 50  0001 L CNN "Arrow Price/Stock"
-	1    4100 3550
-	1    0    0    -1
-$EndComp
-$Comp
 L Device:C C2
 U 1 1 622ECF54
 P 4050 3850
 F 0 "C2" H 4165 3896 50  0000 L CNN
-F 1 "27p" H 4165 3805 50  0000 L CNN
+F 1 "?" H 4165 3805 50  0000 L CNN
 F 2 "" H 4088 3700 50  0001 C CNN
 F 3 "~" H 4050 3850 50  0001 C CNN
@@
 P 4950 3850
 F 0 "C5" H 5065 3896 50  0000 L CNN
-F 1 "27p" H 5065 3805 50  0000 L CNN
+F 1 "?" H 5065 3805 50  0000 L CNN
 F 2 "" H 4988 3700 50  0001 C CNN
 F 3 "~" H 4950 3850 50  0001 C CNN
@@
 $EndComp
 Wire Wire Line
-	4100 3550 4050 3550
-Wire Wire Line
 	4050 3550 4050 3700
 Wire Wire Line
-	4800 3550 4950 3550
-Wire Wire Line
 	4950 3550 4950 3700
 Wire Wire Line
 	4050 4000 4050 4050
 Wire Wire Line
-	4050 4050 4550 4050
+	4050 4050 4450 4050
 Wire Wire Line
 	4550 4050 4950 4050
@@
 $EndComp
 $Comp
-L Flash_memory:W25Q16JVUXIQ U?
+L PSE_RP2040-rescue:W25Q16JVUXIQ-Flash_memory U?
 U 1 1 62321CDF
 P 13450 3200
@@
 	14150 7750 14150 7900
 $Comp
-L gpsChip:PAM7Q U?
+L PSE_RP2040-rescue:PAM7Q-gpsChip U?
 U 1 1 62557D93
 P 14450 9250
@@
 GPIO25
 $Comp
-L buck_converter:RT6150A_B U?
+L PSE_RP2040-rescue:RT6150A_B-buck_converter U?
 U 1 1 62858E49
 P 2200 8850
@@
 Wire Notes Line
 	500  4500 16050 4500
+$Comp
+L Device:Crystal_GND24 Y?
+U 1 1 6234C592
+P 4450 3550
+F 0 "Y?" H 4644 3596 50  0000 L CNN
+F 1 "Crystal_GND24" H 4644 3505 50  0000 L CNN
+F 2 "" H 4450 3550 50  0001 C CNN
+F 3 "~" H 4450 3550 50  0001 C CNN
+	1    4450 3550
+	1    0    0    -1
+$EndComp
+Wire Wire Line
+	4600 3550 4950 3550
+Wire Wire Line
+	4050 3550 4300 3550
+Wire Wire Line
+	4450 3350 4450 3750
+Wire Wire Line
+	4450 3750 4450 4050
+Connection ~ 4450 3750
+Connection ~ 4450 4050
+Wire Wire Line
+	4450 4050 4550 4050
 $EndSCHEMATC
