File: PSE_RP2040/PSE_RP2040.kicad_pcb (KiCad board)
At the start: 2 copper layers, 85 x 56 mm, 129 parts, among them IC1 LAN8742A-CZ, IC2 SAM-M8Q-0, J1 USB_B, J2 USB_B_Mini, J3 8P8C_LED, J4 Conn_01x03, J5 Screw_Terminal_01x02, J6 Conn_01x04_Female, Q2 IRLML6402, SW1 SW_Push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

Commit message: Gerber controllati
Parts:
- moved FID3 21.7 mm to (174.9, 130.5)
- moved Y1 2.48 mm to (183.1, 130.0), turned to 180 degrees
- moved R31 0.20 mm to (145.0, 155.9)
- moved R29 0.20 mm to (146.6, 155.9)
Routing:
- net /VUSB: track 24.1 -> 18.2 mm, vias 0 -> 1
- net GND: track 33.6 -> 38.8 mm, vias 52 -> 51
- net Net-(U2-Pad1): track 6.50 -> 2.69 mm
- net Net-(JP1-Pad2): track 9.11 -> 10.8 mm
- net +3V3: track 203.4 -> 204.7 mm
- net Net-(U2-Pad2): track 3.58 -> 2.54 mm
- net poe+: track 50.9 -> 49.9 mm
- net Net-(IC1-Pad23): track 30.2 -> 29.4 mm
- net Net-(R30-Pad1): track 10.0 -> 10.6 mm
- net Net-(R11-Pad2): vias 0 -> 1
Other:
- board text added: "BOOT"
- board text added: "ERRORI: 11 AVVISI: 8 TESTPOINT TP1 3V3 TP2 GND TP3 5V TP4 1V1 TP5 POE+ TP6 POE- TP7 USB_DP TP8 USB_DN TP9 UART_TX-GPS_RX TP10 UART_RX-GPS_TX TP11 VCC_GPS TP12 GPIO3_I2C_SCL TP13 GPIO2_I2C_SDA"
- board text added: "PPSE2021_LAN_NTP P.A. 209926 P.G. 209048 T.E. 209212 A.M. 209615 T.G. 209359"
- board text added: "RESET"
- board text added: "UNITN"
- board text removed: ">Errori ridotti a 11"
- board text removed: "ERRORI: 11 AVVISI: 6 TESTPOINT TP1 3V3 TP2 GND TP3 5V TP4 1V1 TP5 POE+ TP6 POE- TP7 USB_DP TP8 USB_DN TP9 UART_TX-GPS_RX TP10 UART_RX-GPS_TX TP11 VCC_GPS TP12 GPIO3_I2C_SCL TP13 GPIO2_I2C_SDA"
- board text removed: "PPE2021_LAN_NTP P.A. 209926 P.G. 209048 T.E. 209212 A.M. 209615 T.G. 209359"
- board text removed: "footprint Rpi4"
