File: PSE_RP2040/lan.kicad_sch (KiCad schematic)
At the start: 32 parts, among them IC1 LAN8742A-CZ, T1 749013011, U4 USBLC6-4SC6, Y3 25MHz

Commit message: Gerber controllati
Other:
- title: (none) -> PPSE_LAN_NTP
Changed lines of the file:
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@@
 (kicad_sch (version 20211123) (generator eeschema)
   (paper "A4")
+  (title_block
+    (title "PPSE_LAN_NTP")
+    (date "2022-04-12")
+    (rev "0")
+  )
   (junction (at 121.92 63.5) (diameter 0) (color 0 0 0 0)
   )

Commit message: inseriti valori mancanti
Parts:
- L2: value 25uH -> (none)
Other:
- note removed: "ft = 100KHz"
Changed lines of the file:
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@@
     (stroke (width 0) (type default) (color 0 0 0 0))
-  )
-  (text "ft =  100KHz\n" (at 181.61 59.69 0)
-    (effects (font (size 1.27 1.27)) (justify left bottom))
   )
   (global_label "MDC" (shape input) (at 91.44 132.08 270) (fields_autoplaced)
@@
   (symbol (lib_id "Device:L") (at 173.99 57.15 0) (unit 1)
     (in_bom yes) (on_board yes) (fields_autoplaced)
-    (property "Reference" "L2" (id 0) (at 175.26 55.8799 0)
-      (effects (font (size 1.27 1.27)) (justify left))
-    )
-    (property "Value" "25uH" (id 1) (at 175.26 58.4199 0)
-      (effects (font (size 1.27 1.27)) (justify left))
-    )
+    (property "Reference" "L2" (id 0) (at 175.26 56.3153 0)
+      (effects (font (size 1.27 1.27)) (justify left))
+    )
+    (property "Value" "" (id 1) (at 175.26 58.8522 0)
+      (effects (font (size 1.27 1.27)) (justify left))
+    )
